File: KeebCard/KeebCard.kicad_pcb (KiCad board)
At the start: 2 copper layers, 61 x 36.8 mm, 15 parts, among them J1 Conn_02x03_Odd_Even, SW1 SW_Push, SW2 SW_Push, SW3 SW_Push, U1 ATTINY85-20SU

Commit message: Last minute PCB changes
Parts:
- BT1: footprint bobness_card:SMTU2032 -> KeebCard:SMTU2032
- DS1: footprint bobness_card:SSD1306_OLED_Display_128x32 -> KeebCard:SSD1306_OLED_Display_128x32
- SW1, SW2, SW3: footprint bobness_card:CHERRY_CHOC_PCB -> KeebCard:CHERRY_CHOC_PCB
- U1: footprint bobness_card:ATTINY85-20SU -> KeebCard:ATTINY85-20SU
